File: outputs/amiga_scandoubler/hardware/amiga_scandoubler_v030wip.kicad_pcb (KiCad board)
At the start: 4 copper layers, 95 x 95 mm, 135 parts, among them J1 33DSMT1-E15SNCT, J2 33DSMT1-E15SNCT, J3 TYPE-C-31-M-12, J4 JTAG 2x05 2.54mm, U1 TVP7002PZP, U2 GW1N-LV4QN88C6/I5, U3 ADV7125KSTZ140, U4 SN74LVC2G17DBVR, U5 SN74LVC2G17DBVR, U6 SN74LVC1G17DBVR, U7 TPS62160DSGR, U8 TPS62160DSGR, U9 TPS62160DSGR, Y1 27MHz ECS-3225MVLC

Commit message: v0.31 DAC 再ピン: U2→U3 を交差なしにするピン割当へ変更
- 出力用 28 ピン(3,13-20,25-42,47)を U3 の周回順に合わせて再割当
  R0=47, R1-7=42-36, G0-7=35-28, BLANK=27, B0/1=26/25, B2-7=20-15,
  H_OUT=14, V_OUT=13, DAC_CLK=3
- constraints/amiga_board_top_v031dac.cst を追加し amiga_board_top.cst を更新
- 基板の U2 パッドネットを書き換え(DRC エラー 0、未接続 78 で変化なし)
- YoWASP yosys/nextpnr で P&R: 1816/2048 とも全クロック PASS、phase180 検査 PASS
  DAC 出力の抽出遅延(推定)は最大 3.93/4.25ns(半周期 8.81ns に対し余裕)
- 結果とログを work/v031dac/fpga/ に保存

Co-Authored-By: Claude Opus 5.5 <noreply@anthropic.com>
Claude-Session: https://claude.ai/code/session_019f929sAJ7LRnJRRFvA6g9F
Connections:
- U2 pad 13: H_OUT_RAW -> V_OUT_RAW
- U2 pad 14: V_OUT_RAW -> H_OUT_RAW
- U2 pad 15: DAC_BLANK_N -> DAC_B7
- U2 pad 16: DAC_CLK_RAW -> DAC_B6
- U2 pad 17: DAC_R0 -> DAC_B5
- U2 pad 18: DAC_R1 -> DAC_B4
- U2 pad 19: DAC_R2 -> DAC_B3
- U2 pad 20: DAC_R3 -> DAC_B2
- U2 pad 25: DAC_R4 -> DAC_B1
- U2 pad 26: DAC_R5 -> DAC_B0
- U2 pad 27: DAC_R6 -> DAC_BLANK_N
- U2 pad 28: DAC_R7 -> DAC_G7
- U2 pad 29: DAC_G0 -> DAC_G6
- U2 pad 3: DAC_B7 -> DAC_CLK_RAW
- U2 pad 30: DAC_G1 -> DAC_G5
- U2 pad 31: DAC_G2 -> DAC_G4
- U2 pad 33: DAC_G4 -> DAC_G2
- U2 pad 34: DAC_G5 -> DAC_G1
- U2 pad 35: DAC_G6 -> DAC_G0
- U2 pad 36: DAC_G7 -> DAC_R7
- U2 pad 37: DAC_B0 -> DAC_R6
- U2 pad 38: DAC_B1 -> DAC_R5
- U2 pad 39: DAC_B2 -> DAC_R4
- U2 pad 40: DAC_B3 -> DAC_R3
- U2 pad 41: DAC_B4 -> DAC_R2
- U2 pad 42: DAC_B5 -> DAC_R1
- U2 pad 47: DAC_B6 -> DAC_R0
Changed lines of the file:
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@@
       (net 43 "GND") (solder_mask_margin 0.025))
     (pad "3" smd roundrect (at -4.95 -3.4 180) (size 0.85 0.2) (layers "F.Cu" "F.Paste" "F.Mask") (roundrect_rratio 0.25)
-      (net 88 "DAC_B7") (solder_mask_margin 0.025))
+      (net 96 "DAC_CLK_RAW") (solder_mask_margin 0.025))
     (pad "4" smd roundrect (at -4.95 -3 180) (size 0.85 0.2) (layers "F.Cu" "F.Paste" "F.Mask") (roundrect_rratio 0.25)
       (net 89 "JTAGSEL_N") (solder_mask_margin 0.025))
@@
       (net 54 "3V3") (solder_mask_margin 0.025))
     (pad "13" smd roundrect (at -4.95 0.6 180) (size 0.85 0.2) (layers "F.Cu" "F.Paste" "F.Mask") (roundrect_rratio 0.25)
+      (net 63 "V_OUT_RAW") (solder_mask_margin 0.025))
+    (pad "14" smd roundrect (at -4.95 1 180) (size 0.85 0.2) (layers "F.Cu" "F.Paste" "F.Mask") (roundrect_rratio 0.25)
       (net 62 "H_OUT_RAW") (solder_mask_margin 0.025))
-    (pad "14" smd roundrect (at -4.95 1 180) (size 0.85 0.2) (layers "F.Cu" "F.Paste" "F.Mask") (roundrect_rratio 0.25)
-      (net 63 "V_OUT_RAW") (solder_mask_margin 0.025))
     (pad "15" smd roundrect (at -4.95 1.4 180) (size 0.85 0.2) (layers "F.Cu" "F.Paste" "F.Mask") (roundrect_rratio 0.25)
-      (net 61 "DAC_BLANK_N") (solder_mask_margin 0.025))
+      (net 88 "DAC_B7") (solder_mask_margin 0.025))
     (pad "16" smd roundrect (at -4.95 1.8 180) (size 0.85 0.2) (layers "F.Cu" "F.Paste" "F.Mask") (roundrect_rratio 0.25)
-      (net 96 "DAC_CLK_RAW") (solder_mask_margin 0.025))
+      (net 87 "DAC_B6") (solder_mask_margin 0.025))
     (pad "17" smd roundrect (at -4.95 2.2 180) (size 0.85 0.2) (layers "F.Cu" "F.Paste" "F.Mask") (roundrect_rratio 0.25)
-      (net 65 "DAC_R0") (solder_mask_margin 0.025))
+      (net 86 "DAC_B5") (solder_mask_margin 0.025))
     (pad "18" smd roundrect (at -4.95 2.6 180) (size 0.85 0.2) (layers "F.Cu" "F.Paste" "F.Mask") (roundrect_rratio 0.25)
-      (net 66 "DAC_R1") (solder_mask_margin 0.025))
+      (net 85 "DAC_B4") (solder_mask_margin 0.025))
     (pad "19" smd roundrect (at -4.95 3 180) (size 0.85 0.2) (layers "F.Cu" "F.Paste" "F.Mask") (roundrect_rratio 0.25)
-      (net 67 "DAC_R2") (solder_mask_margin 0.025))
+      (net 84 "DAC_B3") (solder_mask_margin 0.025))
     (pad "20" smd roundrect (at -4.95 3.4 180) (size 0.85 0.2) (layers "F.Cu" "F.Paste" "F.Mask") (roundrect_rratio 0.25)
-      (net 68 "DAC_R3") (solder_mask_margin 0.025))
+      (net 83 "DAC_B2") (solder_mask_margin 0.025))
     (pad "21" smd roundrect (at -4.95 3.8 180) (size 0.85 0.2) (layers "F.Cu" "F.Paste" "F.Mask") (roundrect_rratio 0.25)
       (net 43 "GND") (solder_mask_margin 0.025))
@@
       (net 43 "GND") (solder_mask_margin 0.025))
     (pad "25" smd roundrect (at -3.4 4.95 180) (size 0.2 0.85) (layers "F.Cu" "F.Paste" "F.Mask") (roundrect_rratio 0.25)
-      (net 69 "DAC_R4") (solder_mask_margin 0.025))
+      (net 82 "DAC_B1") (solder_mask_margin 0.025))
     (pad "26" smd roundrect (at -3 4.95 180) (size 0.2 0.85) (layers "F.Cu" "F.Paste" "F.Mask") (roundrect_rratio 0.25)
-      (net 70 "DAC_R5") (solder_mask_margin 0.025))
+      (net 81 "DAC_B0") (solder_mask_margin 0.025))
     (pad "27" smd roundrect (at -2.6 4.95 180) (size 0.2 0.85) (layers "F.Cu" "F.Paste" "F.Mask") (roundrect_rratio 0.25)
-      (net 71 "DAC_R6") (solder_mask_margin 0.025))
+      (net 61 "DAC_BLANK_N") (solder_mask_margin 0.025))
     (pad "28" smd roundrect (at -2.2 4.95 180) (size 0.2 0.85) (layers "F.Cu" "F.Paste" "F.Mask") (roundrect_rratio 0.25)
-      (net 72 "DAC_R7") (solder_mask_margin 0.025))
+      (net 80 "DAC_G7") (solder_mask_margin 0.025))
     (pad "29" smd roundrect (at -1.8 4.95 180) (size 0.2 0.85) (layers "F.Cu" "F.Paste" "F.Mask") (roundrect_rratio 0.25)
-      (net 73 "DAC_G0") (solder_mask_margin 0.025))
+      (net 79 "DAC_G6") (solder_mask_margin 0.025))
     (pad "30" smd roundrect (at -1.4 4.95 180) (size 0.2 0.85) (layers "F.Cu" "F.Paste" "F.Mask") (roundrect_rratio 0.25)
-      (net 74 "DAC_G1") (solder_mask_margin 0.025))
+      (net 78 "DAC_G5") (solder_mask_margin 0.025))
     (pad "31" smd roundrect (at -1 4.95 180) (size 0.2 0.85) (layers "F.Cu" "F.Paste" "F.Mask") (roundrect_rratio 0.25)
-      (net 75 "DAC_G2") (solder_mask_margin 0.025))
+      (net 77 "DAC_G4") (solder_mask_margin 0.025))
     (pad "32" smd roundrect (at -0.6 4.95 180) (size 0.2 0.85) (layers "F.Cu" "F.Paste" "F.Mask") (roundrect_rratio 0.25)
       (net 76 "DAC_G3") (solder_mask_margin 0.025))
     (pad "33" smd roundrect (at -0.2 4.95 180) (size 0.2 0.85) (layers "F.Cu" "F.Paste" "F.Mask") (roundrect_rratio 0.25)
-      (net 77 "DAC_G4") (solder_mask_margin 0.025))
+      (net 75 "DAC_G2") (solder_mask_margin 0.025))
     (pad "34" smd roundrect (at 0.2 4.95 180) (size 0.2 0.85) (layers "F.Cu" "F.Paste" "F.Mask") (roundrect_rratio 0.25)
-      (net 78 "DAC_G5") (solder_mask_margin 0.025))
+      (net 74 "DAC_G1") (solder_mask_margin 0.025))
     (pad "35" smd roundrect (at 0.6 4.95 180) (size 0.2 0.85) (layers "F.Cu" "F.Paste" "F.Mask") (roundrect_rratio 0.25)
-      (net 79 "DAC_G6") (solder_mask_margin 0.025))
+      (net 73 "DAC_G0") (solder_mask_margin 0.025))
     (pad "36" smd roundrect (at 1 4.95 180) (size 0.2 0.85) (layers "F.Cu" "F.Paste" "F.Mask") (roundrect_rratio 0.25)
-      (net 80 "DAC_G7") (solder_mask_margin 0.025))
+      (net 72 "DAC_R7") (solder_mask_margin 0.025))
     (pad "37" smd roundrect (at 1.4 4.95 180) (size 0.2 0.85) (layers "F.Cu" "F.Paste" "F.Mask") (roundrect_rratio 0.25)
-      (net 81 "DAC_B0") (solder_mask_margin 0.025))
+      (net 71 "DAC_R6") (solder_mask_margin 0.025))
     (pad "38" smd roundrect (at 1.8 4.95 180) (size 0.2 0.85) (layers "F.Cu" "F.Paste" "F.Mask") (roundrect_rratio 0.25)
-      (net 82 "DAC_B1") (solder_mask_margin 0.025))
+      (net 70 "DAC_R5") (solder_mask_margin 0.025))
     (pad "39" smd roundrect (at 2.2 4.95 180) (size 0.2 0.85) (layers "F.Cu" "F.Paste" "F.Mask") (roundrect_rratio 0.25)
-      (net 83 "DAC_B2") (solder_mask_margin 0.025))
+      (net 69 "DAC_R4") (solder_mask_margin 0.025))
     (pad "40" smd roundrect (at 2.6 4.95 180) (size 0.2 0.85) (layers "F.Cu" "F.Paste" "F.Mask") (roundrect_rratio 0.25)
-      (net 84 "DAC_B3") (solder_mask_margin 0.025))
+      (net 68 "DAC_R3") (solder_mask_margin 0.025))
     (pad "41" smd roundrect (at 3 4.95 180) (size 0.2 0.85) (layers "F.Cu" "F.Paste" "F.Mask") (roundrect_rratio 0.25)
-      (net 85 "DAC_B4") (solder_mask_margin 0.025))
+      (net 67 "DAC_R2") (solder_mask_margin 0.025))
     (pad "42" smd roundrect (at 3.4 4.95 180) (size 0.2 0.85) (layers "F.Cu" "F.Paste" "F.Mask") (roundrect_rratio 0.25)
-      (net 86 "DAC_B5") (solder_mask_margin 0.025))
+      (net 66 "DAC_R1") (solder_mask_margin 0.025))
     (pad "43" smd roundrect (at 3.8 4.95 180) (size 0.2 0.85) (layers "F.Cu" "F.Paste" "F.Mask") (roundrect_rratio 0.25)
       (net 43 "GND") (solder_mask_margin 0.025))
@@
       (net 43 "GND") (solder_mask_margin 0.025))
     (pad "47" smd roundrect (at 4.95 3.4 180) (size 0.85 0.2) (layers "F.Cu" "F.Paste" "F.Mask") (roundrect_rratio 0.25)
-      (net 87 "DAC_B6") (solder_mask_margin 0.025))
+      (net 65 "DAC_R0") (solder_mask_margin 0.025))
     (pad "48" smd roundrect (at 4.95 3 180) (size 0.85 0.2) (layers "F.Cu" "F.Paste" "F.Mask") (roundrect_rratio 0.25)
       (net 40 "ADC_R0") (solder_mask_margin 0.025))
