File: outputs/amiga_scandoubler/hardware/01_adc.kicad_sch (KiCad schematic)
At the start: 30 parts, among them U1 TVP7002PZP

Commit message: Select LCSC parts with live JLCPCB stock/price (135 of 139 parts)
- r11_select.py queries JLCPCB's public component search. It matches package and spec (C/V/dielectric, R/tolerance, 0.1% thin film) and ranks basic > preferred > stock.
- Results are in fab/v030wip/parts_selection.csv/.json. r11_apply.py writes LCSC/MPN into the manifest, schematic symbols and netlist.
- Open items:
  - U1 TVP7002: stock 4.
  - J1/J2 CONEC 33DSMT1-E15SNCT: stock 0.
  - Y1 ECS-3225MVLC-270: stock 4. YXC OT2EL4C4JI-111OLP-27M (C5203549) is a datasheet-checked drop-in candidate.
- Nets unchanged (595 nodes match the board). The audit passes. Nothing ordered.

Co-Authored-By: Claude Opus 5.5 <noreply@anthropic.com>
Claude-Session: https://claude.ai/code/session_019f929sAJ7LRnJRRFvA6g9F
Parts:
- C1, C13, C14, C15, C16, C17, C18, C19, C20, C21, C22, C23, C24, C25, C26, C27, C28: LCSC (none) -> C14663; MPN 100nF -> CC0603KRX7R9BB104
- C10, C12, C4, C5, C6, C7, C8: LCSC (none) -> C85973; MPN 10nF -> GRM1885C1H103JA01D
- C11, C3, C9: LCSC (none) -> C106246; MPN 1nF -> CC0603JRNPO9BN102
- C2: LCSC (none) -> C576818; MPN 4.7nF -> CC0603JRNPO9BN472
- R1: LCSC (none) -> C22843; MPN 1.5k -> 0603WAF1501T5E
