File: outputs/amiga_scandoubler/hardware/04_connectors.kicad_sch (KiCad schematic)
At the start: 21 parts, among them J1 33DSMT1-E15SNCT, J2 33DSMT1-E15SNCT, U4 SN74LVC2G17DBVR, U5 SN74LVC2G17DBVR, U6 SN74LVC1G17DBVR

Commit message: Select LCSC parts with live JLCPCB stock/price (135 of 139 parts)
- r11_select.py queries JLCPCB's public component search. It matches package and spec (C/V/dielectric, R/tolerance, 0.1% thin film) and ranks basic > preferred > stock.
- Results are in fab/v030wip/parts_selection.csv/.json. r11_apply.py writes LCSC/MPN into the manifest, schematic symbols and netlist.
- Open items:
  - U1 TVP7002: stock 4.
  - J1/J2 CONEC 33DSMT1-E15SNCT: stock 0.
  - Y1 ECS-3225MVLC-270: stock 4. YXC OT2EL4C4JI-111OLP-27M (C5203549) is a datasheet-checked drop-in candidate.
- Nets unchanged (595 nodes match the board). The audit passes. Nothing ordered.

Co-Authored-By: Claude Opus 5.5 <noreply@anthropic.com>
Claude-Session: https://claude.ai/code/session_019f929sAJ7LRnJRRFvA6g9F
Parts:
- C48, C49, C50, C51, C52, C53: LCSC (none) -> C14663; MPN 100nF -> CC0603KRX7R9BB104
- R15, R16, R17: LCSC (none) -> C319466; MPN 75R 0.1% -> AR03BTCX0750
- R18, R20, R22, R23: LCSC (none) -> C23140; MPN 33R -> 0603WAF330JT5E
- R19, R21: LCSC (none) -> C25803; MPN 100k -> 0603WAF1003T5E
- R24: LCSC (none) -> C23345; MPN 22R -> 0603WAF220JT5E
- U4, U5: LCSC (none) -> C19829674
- U6: LCSC (none) -> C7836

Commit message: Replace Y1 with YXC OT2EL4C4JI-111OLP-27M; reselect parts for 2 boards
- Y1: ECS-3225MVLC-270 (LCSC stock 4) -> C5203549, a pin/land-compatible 3225 CMOS oscillator (datasheet checked). Footprint and routing unchanged.
- Selection re-run for a 2-board build (JLCPCB PCBA minimum is 2). U1 is covered (stock 4). J1/J2 carry C3146802 for Global Sourcing.
- All 139 parts now have LCSC numbers.
- Nets still match (595 nodes). DRC errors 0, unconnected 0. The audit passes.

Co-Authored-By: Claude Opus 5.5 <noreply@anthropic.com>
Claude-Session: https://claude.ai/code/session_019f929sAJ7LRnJRRFvA6g9F
Parts:
- J1, J2: LCSC (none) -> C3146802
Changed lines of the file:
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@@
 (property "Datasheet" "" (id 3) (at 85 33.8 0) (effects (font (size 1.0 1.0)) hide))
 (property "MPN" "33DSMT1-E15SNCT" (id 4) (at 85 33.8 0) (effects (font (size 1.0 1.0)) hide))
-(property "LCSC" "" (id 5) (at 85 33.8 0) (effects (font (size 1.0 1.0)) hide))
+(property "LCSC" "C3146802" (id 5) (at 85 33.8 0) (effects (font (size 1.0 1.0)) hide))
 (pin "1")
 (pin "2")
@@
 (property "Datasheet" "" (id 3) (at 285 33.8 0) (effects (font (size 1.0 1.0)) hide))
 (property "MPN" "33DSMT1-E15SNCT" (id 4) (at 285 33.8 0) (effects (font (size 1.0 1.0)) hide))
-(property "LCSC" "" (id 5) (at 285 33.8 0) (effects (font (size 1.0 1.0)) hide))
+(property "LCSC" "C3146802" (id 5) (at 285 33.8 0) (effects (font (size 1.0 1.0)) hide))
 (pin "1")
 (pin "2")

Commit message: Replace J1/J2 with THT HYC06-HDR15B-060 (3-row DE-15 female)
- New footprint DE15_HOAUC_HYC06-HDR15B-060 from the HOAUC drawing
  (rows 3.08/5.06/7.04 mm from edge, 2.29x1.98 pitch, 2x 3.2 mm PTH locks).
- Board: old CONEC SMD footprints and their fan-out removed (jc_rm.py),
  new parts placed (jc_add.py), 10 signals re-routed with router7 (3 vias),
  covered references re-placed (jc_silk.py).
- DRC 0 errors / 0 unconnected, audit PASS, schematic netlist matches
  (570 connected nodes), drill hits match.
- Schematic, netlist, manifest, parts selection (C711364) and all fab
  outputs regenerated; README/revision/CLAUDE.md updated.

Co-Authored-By: Claude Opus 5.5 <noreply@anthropic.com>
Claude-Session: https://claude.ai/code/session_019f929sAJ7LRnJRRFvA6g9F
Parts:
- J1, J2: value 33DSMT1-E15SNCT -> HYC06-HDR15B-060; footprint Amiga:DE15_Conec_33DSMT1-E15SNCT -> Amiga:DE15_HOAUC_HYC06-HDR15B-060; LCSC C3146802 -> C711364; MPN 33DSMT1-E15SNCT -> HYC06-HDR15B-060
Changed lines of the file:
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@@
 (symbol (lib_id "Amiga:DE15_Female") (at 85 38 0) (unit 1) (in_bom yes) (on_board yes)
 (property "Reference" "J1" (id 0) (at 85 31 0) (effects (font (size 1.0 1.0)) ))
-(property "Value" "33DSMT1-E15SNCT" (id 1) (at 85 33.8 0) (effects (font (size 1.0 1.0)) ))
-(property "Footprint" "Amiga:DE15_Conec_33DSMT1-E15SNCT" (id 2) (at 85 33.8 0) (effects (font (size 1.0 1.0)) hide))
+(property "Value" "HYC06-HDR15B-060" (id 1) (at 85 33.8 0) (effects (font (size 1.0 1.0)) ))
+(property "Footprint" "Amiga:DE15_HOAUC_HYC06-HDR15B-060" (id 2) (at 85 33.8 0) (effects (font (size 1.0 1.0)) hide))
 (property "Datasheet" "" (id 3) (at 85 33.8 0) (effects (font (size 1.0 1.0)) hide))
-(property "MPN" "33DSMT1-E15SNCT" (id 4) (at 85 33.8 0) (effects (font (size 1.0 1.0)) hide))
-(property "LCSC" "C3146802" (id 5) (at 85 33.8 0) (effects (font (size 1.0 1.0)) hide))
+(property "MPN" "HYC06-HDR15B-060" (id 4) (at 85 33.8 0) (effects (font (size 1.0 1.0)) hide))
+(property "LCSC" "C711364" (id 5) (at 85 33.8 0) (effects (font (size 1.0 1.0)) hide))
 (pin "1")
 (pin "2")
@@
 (symbol (lib_id "Amiga:DE15_Female") (at 285 38 0) (unit 1) (in_bom yes) (on_board yes)
 (property "Reference" "J2" (id 0) (at 285 31 0) (effects (font (size 1.0 1.0)) ))
-(property "Value" "33DSMT1-E15SNCT" (id 1) (at 285 33.8 0) (effects (font (size 1.0 1.0)) ))
-(property "Footprint" "Amiga:DE15_Conec_33DSMT1-E15SNCT" (id 2) (at 285 33.8 0) (effects (font (size 1.0 1.0)) hide))
+(property "Value" "HYC06-HDR15B-060" (id 1) (at 285 33.8 0) (effects (font (size 1.0 1.0)) ))
+(property "Footprint" "Amiga:DE15_HOAUC_HYC06-HDR15B-060" (id 2) (at 285 33.8 0) (effects (font (size 1.0 1.0)) hide))
 (property "Datasheet" "" (id 3) (at 285 33.8 0) (effects (font (size 1.0 1.0)) hide))
-(property "MPN" "33DSMT1-E15SNCT" (id 4) (at 285 33.8 0) (effects (font (size 1.0 1.0)) hide))
-(property "LCSC" "C3146802" (id 5) (at 285 33.8 0) (effects (font (size 1.0 1.0)) hide))
+(property "MPN" "HYC06-HDR15B-060" (id 4) (at 285 33.8 0) (effects (font (size 1.0 1.0)) hide))
+(property "LCSC" "C711364" (id 5) (at 285 33.8 0) (effects (font (size 1.0 1.0)) hide))
 (pin "1")
 (pin "2")
@@
 (sheet_instances (path "/" (page "5")))
 (symbol_instances
-(path "/d7285cc1-01a7-52b5-b1b4-a16a6a4410c1/ae09b796-6f50-5fe7-9c95-b0a4ec14b086/90d16bad-4ea0-59e8-a923-94a42cbba873" (reference "J1") (unit 1) (value "33DSMT1-E15SNCT") (footprint "Amiga:DE15_Conec_33DSMT1-E15SNCT"))
-(path "/d7285cc1-01a7-52b5-b1b4-a16a6a4410c1/ae09b796-6f50-5fe7-9c95-b0a4ec14b086/98d74ea0-59ee-58e7-9b24-a838edc2f968" (reference "J2") (unit 1) (value "33DSMT1-E15SNCT") (footprint "Amiga:DE15_Conec_33DSMT1-E15SNCT"))
+(path "/d7285cc1-01a7-52b5-b1b4-a16a6a4410c1/ae09b796-6f50-5fe7-9c95-b0a4ec14b086/90d16bad-4ea0-59e8-a923-94a42cbba873" (reference "J1") (unit 1) (value "HYC06-HDR15B-060") (footprint "Amiga:DE15_HOAUC_HYC06-HDR15B-060"))
+(path "/d7285cc1-01a7-52b5-b1b4-a16a6a4410c1/ae09b796-6f50-5fe7-9c95-b0a4ec14b086/98d74ea0-59ee-58e7-9b24-a838edc2f968" (reference "J2") (unit 1) (value "HYC06-HDR15B-060") (footprint "Amiga:DE15_HOAUC_HYC06-HDR15B-060"))
 (path "/d7285cc1-01a7-52b5-b1b4-a16a6a4410c1/ae09b796-6f50-5fe7-9c95-b0a4ec14b086/24a8cbf1-faad-57b5-a6c7-9501bbe52b13" (reference "R15") (unit 1) (value "75R 0.1%") (footprint "Resistor_SMD:R_0603_1608Metric"))
 (path "/d7285cc1-01a7-52b5-b1b4-a16a6a4410c1/ae09b796-6f50-5fe7-9c95-b0a4ec14b086/927af2e4-add9-5d41-9421-dc8269aded81" (reference "C48") (unit 1) (value "100nF") (footprint "Capacitor_SMD:C_0603_1608Metric"))
