File: outputs/amiga_scandoubler/hardware/05_power.kicad_sch (KiCad schematic)
At the start: 26 parts, among them J3 TYPE-C-31-M-12, U7 TPS62160DSGR, U8 TPS62160DSGR, U9 TPS62160DSGR

Commit message: Select LCSC parts with live JLCPCB stock/price (135 of 139 parts)
- r11_select.py queries JLCPCB's public component search. It matches package and spec (C/V/dielectric, R/tolerance, 0.1% thin film) and ranks basic > preferred > stock.
- Results are in fab/v030wip/parts_selection.csv/.json. r11_apply.py writes LCSC/MPN into the manifest, schematic symbols and netlist.
- Open items:
  - U1 TVP7002: stock 4.
  - J1/J2 CONEC 33DSMT1-E15SNCT: stock 0.
  - Y1 ECS-3225MVLC-270: stock 4. YXC OT2EL4C4JI-111OLP-27M (C5203549) is a datasheet-checked drop-in candidate.
- Nets unchanged (595 nodes match the board). The audit passes. Nothing ordered.

Co-Authored-By: Claude Opus 5.5 <noreply@anthropic.com>
Claude-Session: https://claude.ai/code/session_019f929sAJ7LRnJRRFvA6g9F
Parts:
- C54: LCSC (none) -> C15850; MPN 10uF -> CL21A106KAYNNNE
- C55, C57, C59: LCSC (none) -> C15850; MPN 10uF 10V -> CL21A106KAYNNNE
- C56, C58, C60: LCSC (none) -> C45783; MPN 22uF 10V -> CL21A226MAQNNNE
- F1: LCSC (none) -> C269119; MPN 1A hold - select -> SMD1206B110TFT
- R25, R26: LCSC (none) -> C23186; MPN 5.1k 1% -> 0603WAF5101T5E
- R27: LCSC (none) -> C861315; MPN 312k 0.1% -> RT0603BRD07312KL
- R28, R30, R32: LCSC (none) -> C122538; MPN 100k 0.1% -> RT0603BRD07100KL
- R29: LCSC (none) -> C861114; MPN 137k 0.1% -> RT0603BRD07137KL
- R31: LCSC (none) -> C705780; MPN 49.9k 0.1% -> RT0603BRD0749K9L
- R33, R34: LCSC (none) -> C25804; MPN 10k -> 0603WAF1002T5E
- R35: LCSC (none) -> C25803; MPN 100k -> 0603WAF1003T5E
- U7, U8, U9: LCSC (none) -> C324077

Commit message: ERC: add PWR_FLAG to 9 supply nets, record U3 IO*_N exclusion; ERC clean after exclusions
Co-Authored-By: Claude Opus 5.5 <noreply@anthropic.com>
Claude-Session: https://claude.ai/code/session_019f929sAJ7LRnJRRFvA6g9F
Other:
- note added: "PWR_FLAG: supplies reach these nets through L / FB / fuse (no power-output pin). ERC only."
Changed lines of the file:
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@@
 (text "1V2 enable follows 3V3 PG: VCCX/VCCIO rise before FPGA core." (at 20 266 0) (effects (font (size 1.2 1.2)) (justify left top)))
 (text "USB charging source only; PC USB-A bus power is not supported." (at 20 275 0) (effects (font (size 1.2 1.2)) (justify left top)))
+(global_label "5V" (shape passive) (at 50.8 256.54 180) (effects (font (size 0.9 0.9)) (justify right)))
+(symbol (lib_id "power:PWR_FLAG") (at 50.8 256.54 0) (unit 1) (in_bom yes) (on_board yes)
+(property "Reference" "#FLG01" (id 0) (at 50.8 254.635 0) (effects (font (size 1.27 1.27)) hide))
+(property "Value" "PWR_FLAG" (id 1) (at 50.8 252.73 0) (effects (font (size 1.0 1.0))))
+(property "Footprint" "" (id 2) (at 50.8 256.54 0) (effects (font (size 1.27 1.27)) hide))
+(property "Datasheet" "~" (id 3) (at 50.8 256.54 0) (effects (font (size 1.27 1.27)) hide))
+(pin "1")
+)
+(global_label "3V3" (shape passive) (at 83.82 256.54 180) (effects (font (size 0.9 0.9)) (justify right)))
+(symbol (lib_id "power:PWR_FLAG") (at 83.82 256.54 0) (unit 1) (in_bom yes) (on_board yes)
+(property "Reference" "#FLG02" (id 0) (at 83.82 254.635 0) (effects (font (size 1.27 1.27)) hide))
+(property "Value" "PWR_FLAG" (id 1) (at 83.82 252.73 0) (effects (font (size 1.0 1.0))))
+(property "Footprint" "" (id 2) (at 83.82 256.54 0) (effects (font (size 1.27 1.27)) hide))
+(property "Datasheet" "~" (id 3) (at 83.82 256.54 0) (effects (font (size 1.27 1.27)) hide))
+(pin "1")
+)
+(global_label "1V9" (shape passive) (at 116.84 256.54 180) (effects (font (size 0.9 0.9)) (justify right)))
+(symbol (lib_id "power:PWR_FLAG") (at 116.84 256.54 0) (unit 1) (in_bom yes) (on_board yes)
+(property "Reference" "#FLG03" (id 0) (at 116.84 254.635 0) (effects (font (size 1.27 1.27)) hide))
+(property "Value" "PWR_FLAG" (id 1) (at 116.84 252.73 0) (effects (font (size 1.0 1.0))))
+(property "Footprint" "" (id 2) (at 116.84 256.54 0) (effects (font (size 1.27 1.27)) hide))
+(property "Datasheet" "~" (id 3) (at 116.84 256.54 0) (effects (font (size 1.27 1.27)) hide))
+(pin "1")
+)
+(global_label "1V2" (shape passive) (at 149.86 256.54 180) (effects (font (size 0.9 0.9)) (justify right)))
+(symbol (lib_id "power:PWR_FLAG") (at 149.86 256.54 0) (unit 1) (in_bom yes) (on_board yes)
+(property "Reference" "#FLG04" (id 0) (at 149.86 254.635 0) (effects (font (size 1.27 1.27)) hide))
+(property "Value" "PWR_FLAG" (id 1) (at 149.86 252.73 0) (effects (font (size 1.0 1.0))))
+(property "Footprint" "" (id 2) (at 149.86 256.54 0) (effects (font (size 1.27 1.27)) hide))
+(property "Datasheet" "~" (id 3) (at 149.86 256.54 0) (effects (font (size 1.27 1.27)) hide))
+(pin "1")
+)
+(global_label "ADC_3V3A" (shape passive) (at 182.88 256.54 180) (effects (font (size 0.9 0.9)) (justify right)))
+(symbol (lib_id "power:PWR_FLAG") (at 182.88 256.54 0) (unit 1) (in_bom yes) (on_board yes)
+(property "Reference" "#FLG05" (id 0) (at 182.88 254.635 0) (effects (font (size 1.27 1.27)) hide))
+(property "Value" "PWR_FLAG" (id 1) (at 182.88 252.73 0) (effects (font (size 1.0 1.0))))
+(property "Footprint" "" (id 2) (at 182.88 256.54 0) (effects (font (size 1.27 1.27)) hide))
+(property "Datasheet" "~" (id 3) (at 182.88 256.54 0) (effects (font (size 1.27 1.27)) hide))
+(pin "1")
+)
+(global_label "ADC_1V9A" (shape passive) (at 215.9 256.54 180) (effects (font (size 0.9 0.9)) (justify right)))
+(symbol (lib_id "power:PWR_FLAG") (at 215.9 256.54 0) (unit 1) (in_bom yes) (on_board yes)
+(property "Reference" "#FLG06" (id 0) (at 215.9 254.635 0) (effects (font (size 1.27 1.27)) hide))
+(property "Value" "PWR_FLAG" (id 1) (at 215.9 252.73 0) (effects (font (size 1.0 1.0))))
+(property "Footprint" "" (id 2) (at 215.9 256.54 0) (effects (font (size 1.27 1.27)) hide))
+(property "Datasheet" "~" (id 3) (at 215.9 256.54 0) (effects (font (size 1.27 1.27)) hide))
+(pin "1")
+)
+(global_label "ADC_1V9PLL" (shape passive) (at 248.92 256.54 180) (effects (font (size 0.9 0.9)) (justify right)))
+(symbol (lib_id "power:PWR_FLAG") (at 248.92 256.54 0) (unit 1) (in_bom yes) (on_board yes)
+(property "Reference" "#FLG07" (id 0) (at 248.92 254.635 0) (effects (font (size 1.27 1.27)) hide))
+(property "Value" "PWR_FLAG" (id 1) (at 248.92 252.73 0) (effects (font (size 1.0 1.0))))
+(property "Footprint" "" (id 2) (at 248.92 256.54 0) (effects (font (size 1.27 1.27)) hide))
+(property "Datasheet" "~" (id 3) (at 248.92 256.54 0) (effects (font (size 1.27 1.27)) hide))
+(pin "1")
+)
+(global_label "DAC_3V3" (shape passive) (at 281.94 256.54 180) (effects (font (size 0.9 0.9)) (justify right)))
+(symbol (lib_id "power:PWR_FLAG") (at 281.94 256.54 0) (unit 1) (in_bom yes) (on_board yes)
+(property "Reference" "#FLG08" (id 0) (at 281.94 254.635 0) (effects (font (size 1.27 1.27)) hide))
+(property "Value" "PWR_FLAG" (id 1) (at 281.94 252.73 0) (effects (font (size 1.0 1.0))))
+(property "Footprint" "" (id 2) (at 281.94 256.54 0) (effects (font (size 1.27 1.27)) hide))
+(property "Datasheet" "~" (id 3) (at 281.94 256.54 0) (effects (font (size 1.27 1.27)) hide))
+(pin "1")
+)
+(global_label "GND" (shape passive) (at 314.96 256.54 180) (effects (font (size 0.9 0.9)) (justify right)))
+(symbol (lib_id "power:PWR_FLAG") (at 314.96 256.54 0) (unit 1) (in_bom yes) (on_board yes)
+(property "Reference" "#FLG09" (id 0) (at 314.96 254.635 0) (effects (font (size 1.27 1.27)) hide))
+(property "Value" "PWR_FLAG" (id 1) (at 314.96 252.73 0) (effects (font (size 1.0 1.0))))
+(property "Footprint" "" (id 2) (at 314.96 256.54 0) (effects (font (size 1.27 1.27)) hide))
+(property "Datasheet" "~" (id 3) (at 314.96 256.54 0) (effects (font (size 1.27 1.27)) hide))
+(pin "1")
+)
+(text "PWR_FLAG: supplies reach these nets through L / FB / fuse (no power-output pin). ERC only." (at 50.8 262.89 0) (effects (font (size 1.2 1.2)) (justify left top)))
 (sheet_instances (path "/" (page "6")))
 (symbol_instances
+(path "/d7285cc1-01a7-52b5-b1b4-a16a6a4410c1/9a882110-f218-58d3-9709-ffb02fc976d9/6304eb81-be1a-48b0-91f5-ef90f3165c77" (reference "#FLG01") (unit 1) (value "PWR_FLAG") (footprint ""))
+(path "/d7285cc1-01a7-52b5-b1b4-a16a6a4410c1/9a882110-f218-58d3-9709-ffb02fc976d9/8a693b5d-86a7-4991-88a8-c06e1fe55436" (reference "#FLG02") (unit 1) (value "PWR_FLAG") (footprint ""))
+(path "/d7285cc1-01a7-52b5-b1b4-a16a6a4410c1/9a882110-f218-58d3-9709-ffb02fc976d9/585834bf-bc83-4444-9df3-9d4c34eb3193" (reference "#FLG03") (unit 1) (value "PWR_FLAG") (footprint ""))
+(path "/d7285cc1-01a7-52b5-b1b4-a16a6a4410c1/9a882110-f218-58d3-9709-ffb02fc976d9/8ad631a7-67d4-471d-914d-c9987263366f" (reference "#FLG04") (unit 1) (value "PWR_FLAG") (footprint ""))
+(path "/d7285cc1-01a7-52b5-b1b4-a16a6a4410c1/9a882110-f218-58d3-9709-ffb02fc976d9/8c9a3ecd-dc2c-41b0-81c4-867edc4c2fed" (reference "#FLG05") (unit 1) (value "PWR_FLAG") (footprint ""))
+(path "/d7285cc1-01a7-52b5-b1b4-a16a6a4410c1/9a882110-f218-58d3-9709-ffb02fc976d9/5380dc57-e241-469b-b961-81db6e928c30" (reference "#FLG06") (unit 1) (value "PWR_FLAG") (footprint ""))
+(path "/d7285cc1-01a7-52b5-b1b4-a16a6a4410c1/9a882110-f218-58d3-9709-ffb02fc976d9/26bf478a-a319-4fd4-b08d-1a948594c648" (reference "#FLG07") (unit 1) (value "PWR_FLAG") (footprint ""))
+(path "/d7285cc1-01a7-52b5-b1b4-a16a6a4410c1/9a882110-f218-58d3-9709-ffb02fc976d9/ce85b1da-230f-4c91-af5d-431e401c7d88" (reference "#FLG08") (unit 1) (value "PWR_FLAG") (footprint ""))
+(path "/d7285cc1-01a7-52b5-b1b4-a16a6a4410c1/9a882110-f218-58d3-9709-ffb02fc976d9/ebb094e8-970b-4dfa-b076-399d4881f4df" (reference "#FLG09") (unit 1) (value "PWR_FLAG") (footprint ""))
 (path "/d7285cc1-01a7-52b5-b1b4-a16a6a4410c1/9a882110-f218-58d3-9709-ffb02fc976d9/9c86d4c2-dba3-5db6-999a-5a8ac794a036" (reference "J3") (unit 1) (value "TYPE-C-31-M-12") (footprint "Connector_USB:USB_C_Receptacle_HRO_TYPE-C-31-M-12"))
 (path "/d7285cc1-01a7-52b5-b1b4-a16a6a4410c1/9a882110-f218-58d3-9709-ffb02fc976d9/2a0ffdad-776b-5b9e-aa81-5aeeff5ff3a8" (reference "R25") (unit 1) (value "5.1k 1%") (footprint "Resistor_SMD:R_0603_1608Metric"))

Commit message: JLC DFM/order fixes: move vias off pads, widen J3 slots, re-place silk, replace L1-L3, merge C15850 BOM line
- dfm_vias.py: 31 vias moved (pad gap >= 0.15 mm), via-in-pad removed on C56/C58/C59/C60/C71
- dfm_fix2.py: C71/C29 +0.4 mm, J3 footprint with 0.8 mm slots, C15850 values unified
- dfm_silk.py: 50 reference texts re-placed away from pads/holes
- L1-L3 -> Taiyo Yuden NRS4018T2R2MDGJ (C92959, EasyEDA footprint available)
- DRC 0 errors / 0 unconnected, audit PASS, ERC clean, fab outputs regenerated

Co-Authored-By: Claude Opus 5.5 <noreply@anthropic.com>
Claude-Session: https://claude.ai/code/session_019f929sAJ7LRnJRRFvA6g9F
Parts:
- C54: value 10uF -> 10uF 25V
- C55, C57, C59: value 10uF 10V -> 10uF 25V
- J3: footprint Connector_USB:USB_C_Receptacle_HRO_TYPE-C-31-M-12 -> Amiga:USB_C_Receptacle_HRO_TYPE-C-31-M-12_Slot0.8
- L1, L2, L3: LCSC C7413169 -> C92959; MPN VLS4012CX-2R2M-1 -> NRS4018T2R2MDGJ
